File: STM32 Nucleo Arduino Shield.sch (KiCad schematic (older format))
At the start: 106 parts, among them P1 Power, P2 Analog, P3 Digital, P4 Digital, P5 CONN_1, P6 CONN_1, P7 CONN_1, P8 CONN_1

Commit message: adding a bunch of crap. as usual, evaluation board is getting out of hand
Parts:
- removed P?: CONN_01X03, Pin_Headers:Pin_Header_Straight_1x03, symbol CONN_01X03
- removed U?: STM32F410RBTx, LQFP64, symbol STM32F410RBTx
- added C? (x2): 22μF, Capacitors_SMD:c_elec_5x5.3, symbol CP_US
- added C? (x10): 100n, MyModules:SM0603-C-JRL, symbol C_US
- added D? (x2): S1BB, MyModules:SMB-1C2A, symbol D
- added J? (x5): PJ-301B, MyModules:PJ-301B-JACK-SLOTS, symbol JACK_MONO_SW
- added P?: CONN_02X05, Pin_Headers:Pin_Header_Straight_2x05, symbol CONN_02X05
- added P? (x12): CONN_01X01, symbol CONN_01X01
- added R? (x2): 10, MyModules:SM0805-HAND, symbol R_US
Connections:
- net labels added: AVDD, CLOCK_OUT, DAC_AVDD
- net labels removed: LFO_FREQ_A, LFO_MODE_A, PORTAMENTO_AMNT_A, VCF_CUTOFF_A, VCF_ENV_AMNT_A, VCF_LFO_AMNT_A, VCO1_MOD_A, VCO1_MOD_B, VCO1_MOD_SOURCE_A, VCO1_MOD_SOURCE_B, VCO1_PITCH_A, VCO2_PITCH_A, VCO_MOD_AMNT_A
- wire segments 253 -> 395
- no-connect marks 10 -> 21
Other:
- note added: "DECOUPLING"
- note removed: "Shield for Arduino that uses\nthe same pin disposition\nlike "Uno" board Rev 3."
- moved on the sheet: C?, D?, P1, P2, P3, P4, P5, P6, P7, P8, R?, SW?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

Commit message: footprints assigned, netlist generated, layout started
Parts:
- removed C?: 22p, ~, symbol C_US
- removed C? (x2): 100n, ~, symbol C_US
- removed C?: 0.01µ, MyModules:SM0603-C-JRL, symbol C_US
- removed J? (x3): PJ-301B, MyModules:PJ-301B-JACK-SLOTS, symbol JACK_MONO_SW
- removed P? (x2): CONN_01X01, symbol CONN_01X01
- removed R?: 22K, symbol R_US
- removed R? (x6): 10K, ~, symbol R_US
- removed R?: 22, MyModules:SM0603-R-JRL, symbol R_US
- removed U? (x4): OPA4171, symbol TL074-
- removed U? (x2): CD4051, symbol CD4051
- removed U? (x6): SN7407, symbol SN7407
- removed VR? (x2): 1K, symbol POT_US
- added C32, C33, C34, C35, C36, C37, C38, C39: 0.01µ, MyModules:SM0603-C-JRL, symbol C_US
- added C8: 22p, MyModules:SM0603-C-JRL, symbol C_US
- added J3: PJ-301B, MyModules:PJ-301B-JACK-SLOTS, symbol JACK_MONO_SW
- added P10, P22, P23, P24, P25, P26, P27, P28, P29, P9: CONN_01X01, MyModules:TEST_POINT_5000_SERIES, symbol CONN_01X01
- added R18: 47K, MyModules:SM0603-R-JRL, symbol R_US
- added R22: 220K, MyModules:SM0603-R-JRL, symbol R_US
- added R23, R24: 1K, MyModules:SM0603-R-JRL, symbol R_US
- added R8: 39K, MyModules:SM0603-R-JRL, symbol R_US
- added U1, U12: OPA2171, Housings_SSOP:TSSOP-8_3x3mm_Pitch0.65mm, symbol TL072-
- added U10, U11: TL074-, Housings_SSOP:TSSOP-14_4.4x5mm_Pitch0.65mm, symbol TL074-
- added U6: TS321, TO_SOT_Packages_SMD:SOT-23-5, symbol TS321
- C1, C10, C11, C2, C24, C25, C26, C27, C28, C29, C3, C30, C31, C4, C6, C7, C9: renamed from C?; footprint ~ -> MyModules:SM0603-C-JRL
- C22, C23: renamed from C?; footprint Capacitors_SMD:c_elec_5x5.3 -> MyModules:jrl_c_elec_5x5.3
- C5: renamed from C?; footprint ~ -> MyModules:SM0805-HAND
- D1, D2, D3, D4: renamed from D?; footprint (none) -> MyModules:LED-0805-JRL
- P11, P12, P14, P15, P16, P17, P18, P19, P20, P21: renamed from P?; footprint (none) -> MyModules:TEST_POINT_5000_SERIES
- P13: renamed from P?; footprint Pin_Headers:Pin_Header_Straight_2x05 -> Pin_Headers:Pin_Header_Straight_2x05_Pitch1.27mm
- R1, R10, R11, R12, R13, R14, R2, R25, R3, R4, R5, R6, R9: renamed from R?; footprint ~ -> MyModules:SM0603-R-JRL
- R15, R16, R19, R20: renamed from R?; footprint (none) -> MyModules:SM0603-R-JRL
- R17: renamed from R?; value 22K -> 47K; footprint (none) -> MyModules:SM0603-R-JRL
- R21: renamed from R?; value 68K -> 220K; footprint (none) -> MyModules:SM0603-R-JRL
- R7: renamed from R?; value 68K -> 82k; footprint (none) -> MyModules:SM0603-R-JRL
- SW1: renamed from SW?; footprint (none) -> MyModules:B3F-1050-OMRON
- U2, U3: renamed from U?; footprint ~ -> Housings_SSOP:TSSOP-14_4.4x5mm_Pitch0.65mm
- U4: renamed from U?; footprint (none) -> Housings_SOIC:SOIC-14_3.9x8.7mm_Pitch1.27mm
- U7: renamed from U?; footprint (none) -> Housings_SSOP:TSSOP-16_4.4x5mm_Pitch0.65mm
- U8, U9: renamed from U?; footprint (none) -> MyModules:TSSOP-16_4.4x5mm_Pitch0.65mm_jrl
- VR1: renamed from VR?; footprint (none) -> MyModules:R0904N-SONG-HUEI
- VR2, VR3: renamed from VR?; footprint (none) -> MyModules:TC33X-2
- gave numbers to parts that had none: 23
Connections:
- net CLOCK_OUT is gone; now on an unnamed net: J2.3
- net ~DAC_MUX2_EN is gone; now on net GATE_1: R6.1, U4.12
- net +12V: now also U1.8 (V+), U10.4 (V+), U11.4 (V+), U12.8 (V+), U6.5 (V+); no longer R6.2
- net +3V3: now also C1.1, C40.1, OC1.8, R29.2, U7.4 (DVDD)
- net +5V: now also R6.2; no longer C1.1, C40.1, OC1.8, R29.2, U7.4 (DVDD)
- net -12V: now also U1.4 (V-), U10.11 (V-), U11.11 (V-), U12.4 (V-), U6.2 (V-)
- net CV10: now also C34.1, U10.10 (+)
- net CV11: now also C35.1, U10.12 (+)
- net CV12: now also C36.1, U11.3 (+)
- net CV13: now also C37.1, U11.5 (+)
- net CV14: now also C38.1, U11.10 (+)
- net CV15: now also C39.1, U11.12 (+)
- net CV8: now also C32.1, U10.3 (+)
- net CV9: now also C33.1, U10.5 (+)
- net GND: now also C32.2, C33.2, C34.2, C35.2, C36.2, C37.2, C38.2, C39.2, J3.1, R8.1; no longer R17.2
- net LED0: now also U4.13
- net VDAC1: now also U1.1
- net VDAC2: now also U1.7
- net REF0: now reaches C2.1, R14.1, U7.1 (REFI), U7.16 (REF0)
- net REF0: now also R7.2, P9.1 (P1)
- net at U7.11 (OUT2): now also U12.5 (+)
- net at U7.14 (OUT1): now also U12.3 (+)
- net at U7.3 (OUT0): now also U1.3 (+)
- net at U7.6 (OUT3): now also U1.5 (+)
- net at C7.2, R15.1, R19.2: now also U1.2 (-)
- net at C9.2, R16.1, R20.2: now also U1.6 (-)
- net at R7.1: now also R8.2, U6.3 (+)
- net at C6.2, R17.1, R21.2: now also U12.2 (-)
- net at R21.1: now also R23.1
- net VDAC4: no longer names the net of C6.1
- net VDAC4: now also R23.2, U12.1
- net ~DAC_MUX2: no longer names the net of P4.5 (P5)
- net ~DAC_MUX2: no longer U4.13
- net ~DAC_MUX3: no longer names the net of P3.3 (P3)
- new net: C8.2, R18.1, R22.2, U12.6 (-)
- new net: C8.1, R24.2, U12.7
- new net: J3.3, R22.1, R24.1
- new net: P22.1 (P1), U10.1, U10.2 (-)
- new net: P23.1 (P1), U10.6 (-), U10.7
- new net: P24.1 (P1), U10.8, U10.9 (-)
- new net: P25.1 (P1), U10.13 (-), U10.14
- new net: P26.1 (P1), U11.1, U11.2 (-)
- new net: P27.1 (P1), U11.6 (-), U11.7
- new net: P28.1 (P1), U11.8, U11.9 (-)
- new net: P29.1 (P1), U11.13 (-), U11.14
- new net VREF: P10.1 (P1), R17.2, R18.2, U6.1, U6.4 (-)
- no-connect marks 21 -> 23
Other:
- note removed: "GND through 22R and\ndecoupling C taken\nfrom TR-606 schematic"
- moved on the sheet: C24, C25, C26, C27, C28, C29, C30, C31, C6, C9, D1, D2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

Commit message: more tedious routing
Changed lines of the file:
@@
 F 0 "R1" H 2100 10525 50  0000 C CNN
 F 1 "10K" H 2075 10600 50  0000 C CNN
-F 2 "MyModules:SM0603-R-JRL" H 2200 10525 60  0000 C CNN
+F 2 "MyModules:SM0603-R-JRL" H 2200 10525 60  0001 C CNN
 F 3 "~" H 2200 10525 60  0000 C CNN
 	1    2200 10525

Commit message: mostly routed S&H circuits
Parts:
- P10, P11, P12, P14, P15, P16, P17, P18, P19, P20, P21, P22, P23, P24, P25, P26, P27, P28, P29, P9: footprint MyModules:TEST_POINT_5000_SERIES -> MyModules:TEST_POINT_SMALL
Connections:
- net CV0: now also C26.1, U2.10 (+); no longer C24.1, U2.3 (+)
- net CV10: now also C32.1, U10.3 (+); no longer C34.1, U10.10 (+)
- net CV13: now also C38.1, U11.10 (+); no longer C37.1, U11.5 (+)
- net CV14: now also C37.1, U11.5 (+); no longer C38.1, U11.10 (+)
- net CV2: now also C24.1, U2.3 (+); no longer C26.1, U2.10 (+)
- net CV5: now also C31.1, U3.12 (+); no longer C29.1, U3.5 (+)
- net CV6: now also C29.1, U3.5 (+); no longer C30.1, U3.10 (+)
- net CV7: now also C30.1, U3.10 (+); no longer C31.1, U3.12 (+)
- net CV8: now also C34.1, U10.10 (+); no longer C32.1, U10.3 (+)
Changed lines of the file:
@@
 F 0 "R2" H 2125 11500 50  0000 C CNN
 F 1 "10K" H 2100 11575 50  0000 C CNN
-F 2 "MyModules:SM0603-R-JRL" H 2225 11500 60  0000 C CNN
+F 2 "MyModules:SM0603-R-JRL" H 2225 11500 60  0001 C CNN
 F 3 "~" H 2225 11500 60  0000 C CNN
 	1    2225 11500
@@
 F 0 "R3" H 2125 12450 50  0000 C CNN
 F 1 "10K" H 2100 12525 50  0000 C CNN
-F 2 "MyModules:SM0603-R-JRL" H 2225 12450 60  0000 C CNN
+F 2 "MyModules:SM0603-R-JRL" H 2225 12450 60  0001 C CNN
 F 3 "~" H 2225 12450 60  0000 C CNN
 	1    2225 12450
@@
 F 0 "R4" H 2150 13375 50  0000 C CNN
 F 1 "10K" H 2125 13450 50  0000 C CNN
-F 2 "MyModules:SM0603-R-JRL" H 2250 13375 60  0000 C CNN
+F 2 "MyModules:SM0603-R-JRL" H 2250 13375 60  0001 C CNN
 F 3 "~" H 2250 13375 60  0000 C CNN
 	1    2250 13375
@@
 F 0 "U2" H 14800 5775 60  0000 C CNN
 F 1 "TL074-" H 14900 5375 50  0000 C CNN
-F 2 "Housings_SSOP:TSSOP-14_4.4x5mm_Pitch0.65mm" H 14750 5575 60  0000 C CNN
+F 2 "Housings_SSOP:TSSOP-14_4.4x5mm_Pitch0.65mm" H 14750 5575 60  0001 C CNN
 F 3 "~" H 14750 5575 60  0000 C CNN
 	1    14750 5575
@@
 Text Label 13975 6825 2    60   ~ 0
 CV1
-Text Label 13950 7675 2    60   ~ 0
+Text Label 13975 5675 2    60   ~ 0
 CV2
 Text Label 13950 8625 2    60   ~ 0
@@
 Text Label 13950 10175 2    60   ~ 0
 CV4
+Text Label 14000 13125 2    60   ~ 0
+CV5
 Text Label 13975 11325 2    60   ~ 0
-CV5
+CV6
 Text Label 14000 12175 2    60   ~ 0
-CV6
-Text Label 14000 13125 2    60   ~ 0
 CV7
-Text Label 13975 5675 2    60   ~ 0
+Text Label 13950 7675 2    60   ~ 0
 CV0
 $Comp
@@
 F 0 "P11" H 9625 3600 50  0000 C CNN
 F 1 "CONN_01X01" V 9725 3500 50  0000 C CNN
-F 2 "MyModules:TEST_POINT_5000_SERIES" H 9625 3500 60  0001 C CNN
+F 2 "MyModules:TEST_POINT_SMALL" H 9625 3500 60  0001 C CNN
 F 3 "" H 9625 3500 60  0000 C CNN
 	1    9625 3500
@@
 F 0 "P12" H 9625 5650 50  0000 C CNN
 F 1 "CONN_01X01" V 9725 5550 50  0000 C CNN
-F 2 "MyModules:TEST_POINT_5000_SERIES" H 9625 5550 60  0001 C CNN
+F 2 "MyModules:TEST_POINT_SMALL" H 9625 5550 60  0001 C CNN
 F 3 "" H 9625 5550 60  0000 C CNN
 	1    9625 5550
@@
 F 0 "P14" H 15625 5275 50  0000 C CNN
 F 1 "CONN_01X01" V 15725 5175 50  0000 C CNN
-F 2 "MyModules:TEST_POINT_5000_SERIES" H 15625 5175 60  0001 C CNN
+F 2 "MyModules:TEST_POINT_SMALL" H 15625 5175 60  0001 C CNN
 F 3 "" H 15625 5175 60  0000 C CNN
 	1    15625 5175
@@
 F 0 "P15" H 15625 6425 50  0000 C CNN
 F 1 "CONN_01X01" V 15725 6325 50  0000 C CNN
-F 2 "MyModules:TEST_POINT_5000_SERIES" H 15625 6325 60  0001 C CNN
+F 2 "MyModules:TEST_POINT_SMALL" H 15625 6325 60  0001 C CNN
 F 3 "" H 15625 6325 60  0000 C CNN
 	1    15625 6325
@@
 F 0 "P16" H 15625 7275 50  0000 C CNN
 F 1 "CONN_01X01" V 15725 7175 50  0000 C CNN
-F 2 "MyModules:TEST_POINT_5000_SERIES" H 15625 7175 60  0001 C CNN
+F 2 "MyModules:TEST_POINT_SMALL" H 15625 7175 60  0001 C CNN
 F 3 "" H 15625 7175 60  0000 C CNN
 	1    15625 7175
@@
 F 0 "P17" H 15625 8225 50  0000 C CNN
 F 1 "CONN_01X01" V 15725 8125 50  0000 C CNN
-F 2 "MyModules:TEST_POINT_5000_SERIES" H 15625 8125 60  0001 C CNN
+F 2 "MyModules:TEST_POINT_SMALL" H 15625 8125 60  0001 C CNN
 F 3 "" H 15625 8125 60  0000 C CNN
 	1    15625 8125
@@
 F 0 "P18" H 15625 9775 50  0000 C CNN
 F 1 "CONN_01X01" V 15725 9675 50  0000 C CNN
-F 2 "MyModules:TEST_POINT_5000_SERIES" H 15625 9675 60  0001 C CNN
+F 2 "MyModules:TEST_POINT_SMALL" H 15625 9675 60  0001 C CNN
 F 3 "" H 15625 9675 60  0000 C CNN
 	1    15625 9675
@@
 F 0 "P19" H 15625 10925 50  0000 C CNN
 F 1 "CONN_01X01" V 15725 10825 50  0000 C CNN
-F 2 "MyModules:TEST_POINT_5000_SERIES" H 15625 10825 60  0001 C CNN
+F 2 "MyModules:TEST_POINT_SMALL" H 15625 10825 60  0001 C CNN
 F 3 "" H 15625 10825 60  0000 C CNN
 	1    15625 10825
@@
 F 0 "P20" H 15625 11775 50  0000 C CNN
 F 1 "CONN_01X01" V 15725 11675 50  0000 C CNN
-F 2 "MyModules:TEST_POINT_5000_SERIES" H 15625 11675 60  0001 C CNN
+F 2 "MyModules:TEST_POINT_SMALL" H 15625 11675 60  0001 C CNN
 F 3 "" H 15625 11675 60  0000 C CNN
 	1    15625 11675
@@
 F 0 "P21" H 15625 12725 50  0000 C CNN
 F 1 "CONN_01X01" V 15725 12625 50  0000 C CNN
-F 2 "MyModules:TEST_POINT_5000_SERIES" H 15625 12625 60  0001 C CNN
+F 2 "MyModules:TEST_POINT_SMALL" H 15625 12625 60  0001 C CNN
 F 3 "" H 15625 12625 60  0000 C CNN
 	1    15625 12625
@@
 F 0 "P10" H 5425 7525 50  0000 C CNN
 F 1 "CONN_01X01" V 5525 7425 50  0000 C CNN
-F 2 "MyModules:TEST_POINT_5000_SERIES" H 5425 7425 60  0001 C CNN
+F 2 "MyModules:TEST_POINT_SMALL" H 5425 7425 60  0001 C CNN
 F 3 "" H 5425 7425 60  0000 C CNN
 	1    5425 7425
@@
 F 0 "P9" H 3800 7800 50  0000 C CNN
 F 1 "CONN_01X01" V 3900 7700 50  0000 C CNN
-F 2 "MyModules:TEST_POINT_5000_SERIES" H 3800 7700 60  0001 C CNN
+F 2 "MyModules:TEST_POINT_SMALL" H 3800 7700 60  0001 C CNN
 F 3 "" H 3800 7700 60  0000 C CNN
 	1    3800 7700
@@
 Text Label 16450 6825 2    60   ~ 0
 CV9
-Text Label 16425 7675 2    60   ~ 0
+Text Label 16450 5675 2    60   ~ 0
 CV10
 Text Label 16425 8625 2    60   ~ 0
@@
 Text Label 16425 10175 2    60   ~ 0
 CV12
+Text Label 16475 12175 2    60   ~ 0
+CV13
 Text Label 16450 11325 2    60   ~ 0
-CV13
-Text Label 16475 12175 2    60   ~ 0
 CV14
 Text Label 16475 13125 2    60   ~ 0
 CV15
-Text Label 16450 5675 2    60   ~ 0
+Text Label 16425 7675 2    60   ~ 0
 CV8
 $Comp
@@
 F 0 "P22" H 18100 5275 50  0000 C CNN
 F 1 "CONN_01X01" V 18200 5175 50  0000 C CNN
-F 2 "MyModules:TEST_POINT_5000_SERIES" H 18100 5175 60  0001 C CNN
+F 2 "MyModules:TEST_POINT_SMALL" H 18100 5175 60  0001 C CNN
 F 3 "" H 18100 5175 60  0000 C CNN
 	1    18100 5175
@@
 F 0 "P23" H 18100 6425 50  0000 C CNN
 F 1 "CONN_01X01" V 18200 6325 50  0000 C CNN
-F 2 "MyModules:TEST_POINT_5000_SERIES" H 18100 6325 60  0001 C CNN
+F 2 "MyModules:TEST_POINT_SMALL" H 18100 6325 60  0001 C CNN
 F 3 "" H 18100 6325 60  0000 C CNN
 	1    18100 6325
@@
 F 0 "P24" H 18100 7275 50  0000 C CNN
 F 1 "CONN_01X01" V 18200 7175 50  0000 C CNN
-F 2 "MyModules:TEST_POINT_5000_SERIES" H 18100 7175 60  0001 C CNN
+F 2 "MyModules:TEST_POINT_SMALL" H 18100 7175 60  0001 C CNN
 F 3 "" H 18100 7175 60  0000 C CNN
 	1    18100 7175
@@
 F 0 "P25" H 18100 8225 50  0000 C CNN
 F 1 "CONN_01X01" V 18200 8125 50  0000 C CNN
-F 2 "MyModules:TEST_POINT_5000_SERIES" H 18100 8125 60  0001 C CNN
+F 2 "MyModules:TEST_POINT_SMALL" H 18100 8125 60  0001 C CNN
 F 3 "" H 18100 8125 60  0000 C CNN
 	1    18100 8125
@@
 F 0 "P26" H 18100 9775 50  0000 C CNN
 F 1 "CONN_01X01" V 18200 9675 50  0000 C CNN
-F 2 "MyModules:TEST_POINT_5000_SERIES" H 18100 9675 60  0001 C CNN
+F 2 "MyModules:TEST_POINT_SMALL" H 18100 9675 60  0001 C CNN
 F 3 "" H 18100 9675 60  0000 C CNN
 	1    18100 9675
@@
 F 0 "P27" H 18100 10925 50  0000 C CNN
 F 1 "CONN_01X01" V 18200 10825 50  0000 C CNN
-F 2 "MyModules:TEST_POINT_5000_SERIES" H 18100 10825 60  0001 C CNN
+F 2 "MyModules:TEST_POINT_SMALL" H 18100 10825 60  0001 C CNN
 F 3 "" H 18100 10825 60  0000 C CNN
 	1    18100 10825
@@
 F 0 "P28" H 18100 11775 50  0000 C CNN
 F 1 "CONN_01X01" V 18200 11675 50  0000 C CNN
-F 2 "MyModules:TEST_POINT_5000_SERIES" H 18100 11675 60  0001 C CNN
+F 2 "MyModules:TEST_POINT_SMALL" H 18100 11675 60  0001 C CNN
 F 3 "" H 18100 11675 60  0000 C CNN
 	1    18100 11675
@@
 F 0 "P29" H 18100 12725 50  0000 C CNN
 F 1 "CONN_01X01" V 18200 12625 50  0000 C CNN
-F 2 "MyModules:TEST_POINT_5000_SERIES" H 18100 12625 60  0001 C CNN
+F 2 "MyModules:TEST_POINT_SMALL" H 18100 12625 60  0001 C CNN
 F 3 "" H 18100 12625 60  0000 C CNN
 	1    18100 12625

Commit message: everything placed and routing. stitching ground
Parts:
- P13: footprint Pin_Headers:Pin_Header_Straight_2x05_Pitch1.27mm -> Pin_Headers:Pin_Header_Straight_2x05_Pitch2.54mm
Changed lines of the file:
@@
 F 0 "P13" H 14350 1575 50  0000 C CNN
 F 1 "CONN_02X05" H 14350 975 50  0000 C CNN
-F 2 "Pin_Headers:Pin_Header_Straight_2x05_Pitch1.27mm" H 14350 75  60  0001 C CNN
+F 2 "Pin_Headers:Pin_Header_Straight_2x05_Pitch2.54mm" H 14350 75  60  0001 C CNN
 F 3 "" H 14350 75  60  0000 C CNN
 	1    14350 1275

Commit message: routed. weird Socket_Arduino_Uno library glitch required reinstalling footprint library from Arduino tempalte folder
Parts:
- added P30: CONN_01X01, MyModules:TEST_POINT_SMALL, symbol CONN_01X01
Connections:
- net ANALOG_IN: now reaches P3.9 (P9)
- net ANALOG_IN: now also P30.1 (P1)
- no-connect marks 23 -> 22

Commit message: ready for checking
Parts:
- U6: value TS321 -> OPA171
Connections:
- no-connect marks 22 -> 24
Other:
- moved on the sheet: C1, C10, C11, C12, C13, C14, C15, C16, C17, C18, C19, C2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

Commit message: finished adding 3D models
Parts:
- added P?: CONN_01X01, MyModules:TEST_POINT_LOOP_4592, symbol CONN_01X01
Connections:
- net GND: now also P?.1 (P1)
Changed lines of the file:
@@
 NoConn ~ 9300 8325
 NoConn ~ 10925 8500
+$Comp
+L CONN_01X01 P?
+U 1 1 5899667E
+P 5450 6575
+F 0 "P?" H 5450 6675 50  0000 C CNN
+F 1 "CONN_01X01" V 5550 6575 50  0000 C CNN
+F 2 "MyModules:TEST_POINT_LOOP_4592" H 5450 6575 60  0001 C CNN
+F 3 "" H 5450 6575 60  0000 C CNN
+	1    5450 6575
+	0    -1   -1   0
+$EndComp
+$Comp
+L GND_R #PWR?
+U 1 1 58997933
+P 5450 6775
+F 0 "#PWR?" H 5450 6775 30  0001 C CNN
+F 1 "GND_R" H 5450 6675 30  0001 C CNN
+F 2 "" H 5450 6775 60  0000 C CNN
+F 3 "" H 5450 6775 60  0000 C CNN
+	1    5450 6775
+	1    0    0    -1
+$EndComp
 $EndSCHEMATC
