File: STM32 Nucleo Arduino Shield.kicad_pcb (KiCad board)
At the start: 2 copper layers, 84 x 55.2 mm, 124 parts, among them J1 PJ-301B, J2 PJ-301B, J3 PJ-301B, P1 Power, P10 CONN_01X01, P11 CONN_01X01, P12 CONN_01X01, P13 CONN_02X05, P14 CONN_01X01, P15 CONN_01X01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

Commit message: checked shield footprint and ordered PCBs
Routing:
- net GND: track 51.5 -> 63.1 mm, vias 29 -> 33
Other:
- board text added: "GND"
- board text added: "STM32F410RB NUCLEO MAX5134 EVAL"
- board text added: "r1.0 02 2017"
